File: hardware/hardware.kicad_sch (KiCad schematic)
At the start: 27 parts, among them J2 USB_B_Micro, J3 Conn_01x05_Pin, U1 CH32V003F4P6, U3 AMS1117-3.3

Commit message: fix button
Connections:
- net BUTTON: now also U1.16 (PC6/MOSI)
Other:
- moved on the sheet: D1, D2, D3, D4, D5, D6, R10, R5, R6, R7, R8, R9

Commit message: add code
Changed lines of the file:
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@@
 (kicad_sch
-	(version 20231120)
+	(version 20250114)
 	(generator "eeschema")
-	(generator_version "8.0")
+	(generator_version "9.0")
 	(paper "A4")
+	(text "CONNECTOR"
+		(exclude_from_sim no)
+		(at 16.51 95.25 0)
+		(effects
+			(font
+				(size 1.27 1.27)
+			)
+			(justify left bottom)
+		)
+	)
+	(text "REGULATOR"
+		(exclude_from_sim no)
+		(at 48.26 95.25 0)
+		(effects
+			(font
+				(size 1.27 1.27)
+			)
+			(justify left bottom)
+		)
+	)
 	(junction
 		(at 163.83 99.06)
@@
 		)
 	)
+	(wire
+		(pts
+			(xy 101.6 74.93) (xy 105.41 74.93)
+		)
+		(stroke
+			(width 0)
+			(type default)
+		)
+	)
 	(polyline
 		(pts
@@
 		)
 	)
-	(text "CONNECTOR"
-		(exclude_from_sim no)
-		(at 16.51 95.25 0)
-		(effects
-			(font
-				(size 1.27 1.27)
-			)
-			(justify left bottom)
-		)
-	)
-	(text "REGULATOR"
-		(exclude_from_sim no)
-		(at 48.26 95.25 0)
-		(effects
-			(font
-				(size 1.27 1.27)
-			)
-			(justify left bottom)
-		)
-	)
 	(global_label "BUTTON"
 		(shape input)
@@
 	(symbol
 		(lib_id "power:GND")
-		(at 101.6 74.93 90)
+		(at 105.41 74.93 90)
 		(unit 1)
 		(exclude_from_sim no)
@@
 		(dnp no)
 		(property "Reference" "#PWR09"
-			(at 107.95 74.93 0)
+			(at 111.76 74.93 0)
 			(effects
 				(font
@@
 		)
 		(property "Value" "GND"
-			(at 101.6 77.47 90)
+			(at 105.41 77.47 90)
 			(effects
 				(font
@@
 		)
 		(property "Footprint" ""
-			(at 101.6 74.93 0)
+			(at 105.41 74.93 0)
 			(effects
 				(font
@@
 		)
 		(property "Datasheet" ""
-			(at 101.6 74.93 0)
+			(at 105.41 74.93 0)
 			(effects
 				(font
@@
 		)
 		(property "Description" ""
-			(at 101.6 74.93 0)
+			(at 105.41 74.93 0)
 			(effects
 				(font
@@
 		)
 	)
+	(embedded_fonts no)
 )
